File: m47Board-H503.kicad_pcb (KiCad board)
At the start: 4 copper layers, 40 x 34 mm, 42 parts, among them J1 USB_C_Receptacle_USB2.0_16P, J3 Conn_01x15_Pin, J4 Conn_01x10_Pin, J5 Conn_01x15_Pin, SW1 SW_Push, SW2 SW_Push, SW3 SW_Push, U1 AP2114H-3.3TRG1, U2 STM32H503CBTx, U3 USBLC6-2SC6, Y1 CX3225FB16000F0FZZH1 16MHz, Y2 ABS07-32.768KHZ-T

Commit message: Add copper zones
Connections:
- J1 pad SH: unconnected-(J1-SHIELD-PadSH)_1 -> GND
Routing:
- net /NRST: track 9.61 -> 18.7 mm
- net Net-(R2-Pad2): track 4.18 -> 13.3 mm
- added copper zone on In2.Cu, net +3.3V
- added copper zone on In1.Cu, net GND
- added copper zone on In2.Cu, net VBUS
Changed lines of the file:
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@@
 			(layers "*.Cu" "*.Mask" "F.Paste")
 			(remove_unused_layers no)
-			(net "unconnected-(J1-SHIELD-PadSH)")
+			(net "GND")
 			(pinfunction "SHIELD_SH")
-			(pintype "passive+no_connect")
+			(pintype "passive")
 		)
 		(pad "SH" thru_hole oval
@@
 			(layers "*.Cu" "*.Mask" "F.Paste")
 			(remove_unused_layers no)
-			(net "unconnected-(J1-SHIELD-PadSH)_2")
+			(net "GND")
 			(pinfunction "SHIELD_SH")
-			(pintype "passive+no_connect")
+			(pintype "passive")
 		)
 		(pad "SH" thru_hole oval
@@
 			(layers "*.Cu" "*.Mask" "F.Paste")
 			(remove_unused_layers no)
-			(net "unconnected-(J1-SHIELD-PadSH)_3")
+			(net "GND")
 			(pinfunction "SHIELD_SH")
-			(pintype "passive+no_connect")
+			(pintype "passive")
 		)
 		(pad "SH" thru_hole oval
@@
 			(layers "*.Cu" "*.Mask" "F.Paste")
 			(remove_unused_layers no)
-			(net "unconnected-(J1-SHIELD-PadSH)_1")
+			(net "GND")
 			(pinfunction "SHIELD_SH")
-			(pintype "passive+no_connect")
+			(pintype "passive")
 		)
 		(embedded_fonts no)
@@
 	)
 	(segment
+		(start 139.8 95.93)
+		(end 148.9 95.93)
+		(width 0.2)
+		(layer "F.Cu")
+		(net "Net-(R2-Pad2)")
+	)
+	(segment
 		(start 148.9 95.93)
 		(end 148.9 96.7925)
@@
 	)
 	(segment
+		(start 126.8 95.93)
+		(end 135.9 95.93)
+		(width 0.2)
+		(layer "F.Cu")
+		(net "/NRST")
+	)
+	(segment
 		(start 144.69 102.61)
 		(end 145.2775 102.61)
@@
 		(net "/BOOT0")
 	)
+	(zone
+		(net "GND")
+		(layer "In1.Cu")
+		(hatch edge 0.5)
+		(connect_pads
+			(clearance 0.2)
+		)
+		(min_thickness 0.25)
+		(fill yes
+			(thermal_gap 0.5)
+			(thermal_bridge_width 0.5)
+			(island_removal_mode 0)
+		)
+		(polygon
+			(pts
+				(xy 120 86) (xy 160 86) (xy 160 120) (xy 120 120)
+			)
+		)
+	)
+	(zone
+		(net "+3.3V")
+		(layer "In2.Cu")
+		(hatch edge 0.5)
+		(priority 1)
+		(connect_pads
+			(clearance 0.2)
+		)
+		(min_thickness 0.25)
+		(fill yes
+			(thermal_gap 0.5)
+			(thermal_bridge_width 0.5)
+			(island_removal_mode 0)
+		)
+		(polygon
+			(pts
+				(xy 120 86) (xy 160 86) (xy 160 120) (xy 120 120)
+			)
+		)
+	)
+	(zone
+		(net "VBUS")
+		(layer "In2.Cu")
+		(hatch edge 0.5)
+		(priority 2)
+		(connect_pads
+			(clearance 0.2)
+		)
+		(min_thickness 0.25)
+		(fill yes
+			(thermal_gap 0.5)
+			(thermal_bridge_width 0.5)
+			(island_removal_mode 0)
+		)
+		(polygon
+			(pts
+				(xy 160 93.8) (xy 151.6 93.8) (xy 151.6 108.1) (xy 154.4 108.1) (xy 154.4 113.3) (xy 150.4 113.3)
+				(xy 150.4 115.6) (xy 160 115.6)
+			)
+		)
+	)
 	(embedded_fonts no)

Commit message: Route traces
Parts:
- moved C6 0.24 mm to (134.4, 105.5)
Connections:
- J3 pad 10: unconnected-(J3-Pin_10-Pad10) -> /PB6
- J3 pad 11: unconnected-(J3-Pin_11-Pad11) -> /PB7
- J3 pad 12: unconnected-(J3-Pin_12-Pad12) -> /PB8
- J3 pad 13: unconnected-(J3-Pin_13-Pad13) -> /PC13
- J3 pad 14: unconnected-(J3-Pin_14-Pad14) -> Net-(J3-Pin_14)
- J3 pad 15: unconnected-(J3-Pin_15-Pad15) -> Net-(J3-Pin_15)
- J3 pad 2: /SWCLK -> GND
- J3 pad 3: GND -> /SWDIO
- J3 pad 4: /SWDIO -> /SWCLK
- J3 pad 6: unconnected-(J3-Pin_6-Pad6) -> /PA15
- J3 pad 7: unconnected-(J3-Pin_7-Pad7) -> /PB3
- J3 pad 8: unconnected-(J3-Pin_8-Pad8) -> /PB4
- J3 pad 9: unconnected-(J3-Pin_9-Pad9) -> /PB5
- R6 pad 2: unconnected-(R6-Pad2) -> Net-(J3-Pin_14)
- R7 pad 2: unconnected-(R7-Pad2) -> Net-(J3-Pin_15)
Routing:
- net /PC13: track 3.04 -> 32.0 mm, vias 0 -> 1
- net /SWDIO: track 0.00 -> 18.3 mm, vias 0 -> 1
- net Net-(J3-Pin_15): track 0.00 -> 17.1 mm
- net /PB8: track 0.00 -> 16.0 mm, vias 0 -> 1
- net /PB7: track 0.00 -> 15.4 mm, vias 0 -> 1
- net /NRST: track 18.7 -> 33.4 mm
- net /PB6: track 0.00 -> 14.5 mm, vias 0 -> 1
- net /SWCLK: track 0.41 -> 14.6 mm, vias 0 -> 1
- net /PB5: track 0.00 -> 13.7 mm, vias 0 -> 1
- net Net-(J3-Pin_14): track 0.00 -> 13.0 mm
- net GND: track 5.44 -> 18.4 mm, vias 0 -> 9
- net /PB4: track 0.00 -> 12.8 mm, vias 0 -> 1
- net /PA15: track 0.00 -> 12.7 mm, vias 0 -> 1
- net /PB3: track 0.00 -> 12.0 mm, vias 0 -> 1
- net VBUS: track 6.32 -> 8.16 mm, vias 0 -> 2
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